File: PCB/keyboard-V1.1.kicad_pcb (KiCad board)
At the start: 2 copper layers, 110 x 80 mm, 14 parts, among them SW1 SW_Push, SW10 SW_Push, SW2 SW_Push, SW3 SW_Push, SW4 SW_Push, SW5 SW_Push, SW6 SW_Push, SW7 SW_Push, SW8 SW_Push, SW9 SW_Push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

Commit message: tried to update the skmini thing
itssssss noooooooot workingggggggggggg
Parts:
- removed D1, D2, D3: SK6812MINI, LED_SMD:LED_SK6812MINI_PLCC4_3.5x3.5mm_P1.75mm
- added D7: SK6812MINI-E, LED_SMD:LED_SK6812MINI_PLCC4_3.5x3.5mm_P1.75mm, F.Cu at (160.0, 64.0)
- added D8: SK6812MINI-E, LED_SMD:LED_SK6812MINI_PLCC4_3.5x3.5mm_P1.75mm, F.Cu at (175.0, 64.0)
- added D9: SK6812MINI-E, LED_SMD:LED_SK6812MINI_PLCC4_3.5x3.5mm_P1.75mm, F.Cu at (186.0, 64.0)
Routing:
- net Net-(D8-DOUT): track 0.00 -> 39.5 mm, vias 0 -> 4
- net Net-(D7-DOUT): track 0.00 -> 35.5 mm, vias 0 -> 2
- net Net-(D2-DOUT): track 30.3 -> 0.00 mm
- net Net-(D1-DOUT): track 12.6 -> 0.00 mm, vias 2 -> 0
- net Net-(D7-DIN): track 56.9 -> 48.5 mm, vias 1 -> 2
- net +5V: track 68.4 -> 61.6 mm, vias 0 -> 3
- net GND: track 311.4 -> 308.3 mm, vias 1 -> 7
Other:
- board text added: "Bob's Mini-Keyboard V1.2"
- board text removed: "Bob's Mini-Keyboard V1.1"
